File: pcb/sparc_pcb_v2.kicad_pcb (KiCad board)
At the start: 2 copper layers, 36.5 x 36.5 mm, 22 parts, among them SW4 Reset, SW5 BOOT, U2 ESP32-WROOM-32

Commit message: cleaned up the pcb a bit and made it pass drc
Parts:
- moved C4 0.72 mm to (144.4, 94.6)
Routing:
- net Net-(U2-IO17): track 32.3 -> 14.1 mm
- net Net-(U2-IO16): track 16.1 -> 28.4 mm
- net TP4056 OUT+: track 38.6 -> 49.1 mm
- net GND: vias 0 -> 5
Changed lines of the file:
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@@
 	(footprint "Capacitor_SMD:C_1206_3216Metric_Pad1.33x1.80mm_HandSolder"
 		(layer "F.Cu")
-		(at 145.13 94.6625)
+		(at 144.41 94.58)
 		(descr "Capacitor SMD 1206 (3216 Metric), square (rectangular) end terminal, IPC-7351 nominal with elongated pad for handsoldering. (Body size source: IPC-SM-782 page 76, https://www.pcb-3d.com/wordpress/wp-content/uploads/ipc-sm-782a_amendment_1_and_2.pdf)")
 		(tags "capacitor handsolder")
@@
 		(net "+3.3V")
 	)
+	(via
+		(at 116.79 87.78)
+		(size 0.6)
+		(drill 0.3)
+		(layers "F.Cu" "B.Cu")
+		(free yes)
+		(net "GND")
+	)
+	(via
+		(at 142.25 89.33)
+		(size 0.6)
+		(drill 0.3)
+		(layers "F.Cu" "B.Cu")
+		(free yes)
+		(net "GND")
+	)
+	(via
+		(at 124.74 78.67)
+		(size 0.6)
+		(drill 0.3)
+		(layers "F.Cu" "B.Cu")
+		(free yes)
+		(net "GND")
+	)
+	(via
+		(at 126.14 96.92)
+		(size 0.6)
+		(drill 0.3)
+		(layers "F.Cu" "B.Cu")
+		(free yes)
+		(net "GND")
+	)
+	(via
+		(at 141.55 74.94)
+		(size 0.6)
+		(drill 0.3)
+		(layers "F.Cu" "B.Cu")
+		(free yes)
+		(net "GND")
+	)
+	(segment
+		(start 144.14 97)
+		(end 142.8475 95.7075)
+		(width 0.5)
+		(layer "F.Cu")
+		(net "TP4056 OUT+")
+	)
+	(segment
+		(start 147.07 97)
+		(end 144.14 97)
+		(width 0.5)
+		(layer "F.Cu")
+		(net "TP4056 OUT+")
+	)
 	(segment
 		(start 135.6 105.46)
@@
 	)
 	(segment
-		(start 146.16 91.615908)
-		(end 145.560908 92.215)
-		(width 0.25)
-		(layer "F.Cu")
-		(net "TP4056 OUT+")
-	)
-	(segment
 		(start 146.16 91.2275)
 		(end 146.16 91.615908)
@@
 	)
 	(segment
+		(start 142.8475 95.7075)
+		(end 142.8475 94.58)
+		(width 0.5)
+		(layer "F.Cu")
+		(net "TP4056 OUT+")
+	)
+	(segment
 		(start 123.99 106.67)
 		(end 123.99 105.47)
@@
 	)
 	(segment
-		(start 145.560908 92.215)
-		(end 144.585001 92.215)
-		(width 0.25)
+		(start 146.16 91.2275)
+		(end 148.01 93.0775)
+		(width 0.5)
 		(layer "F.Cu")
 		(net "TP4056 OUT+")
@@
 	)
 	(segment
-		(start 144.585001 92.215)
-		(end 144.26 91.889999)
-		(width 0.25)
+		(start 148.01 96.06)
+		(end 147.07 97)
+		(width 0.5)
+		(layer "F.Cu")
+		(net "TP4056 OUT+")
+	)
+	(segment
+		(start 148.01 93.0775)
+		(end 148.01 96.06)
+		(width 0.5)
 		(layer "F.Cu")
 		(net "TP4056 OUT+")
@@
 	)
 	(segment
-		(start 117.938604 97.175)
-		(end 118.925 98.161396)
+		(start 120 94.79)
+		(end 120 95.5)
 		(width 0.25)
 		(layer "B.Cu")
@@
 	)
 	(segment
-		(start 118.925 98.161396)
-		(end 118.925 99.3701)
+		(start 119 95.5)
+		(end 120 95.5)
 		(width 0.25)
 		(layer "B.Cu")
@@
 	)
 	(segment
-		(start 120.5451 99.7)
-		(end 120.875 99.3701)
+		(start 120.535 87.715)
+		(end 118.78 89.47)
 		(width 0.25)
 		(layer "B.Cu")
@@
 	)
 	(segment
-		(start 115.179968 95.966669)
-		(end 116.388299 97.175)
-		(width 0.25)
-		(layer "B.Cu")
-		(net "Net-(U2-IO17)")
-	)
-	(segment
-		(start 119.2549 99.7)
-		(end 120.5451 99.7)
+		(start 122.275 87.715)
+		(end 120.535 87.715)
 		(width 0.25)
 		(layer "B.Cu")
@@
 	)
 	(segment
-		(start 115.179968 91.033331)
-		(end 115.179968 95.966669)
+		(start 118.78 89.47)
+		(end 118.78 93.57)
 		(width 0.25)
 		(layer "B.Cu")
@@
 	)
 	(segment
-		(start 120.875 99.3701)
-		(end 120.875 97.375)
+		(start 118.78 93.57)
+		(end 120 94.79)
 		(width 0.25)
 		(layer "B.Cu")
@@
 	)
 	(segment
-		(start 118.925 99.3701)
-		(end 119.2549 99.7)
-		(width 0.25)
-		(layer "B.Cu")
-		(net "Net-(U2-IO17)")
-	)
-	(segment
-		(start 120.875 97.375)
-		(end 117 93.5)
-		(width 0.25)
-		(layer "B.Cu")
-		(net "Net-(U2-IO17)")
-	)
-	(segment
-		(start 122.275 87.715)
-		(end 118.498299 87.715)
-		(width 0.25)
-		(layer "B.Cu")
-		(net "Net-(U2-IO17)")
-	)
-	(segment
-		(start 118.498299 87.715)
-		(end 115.179968 91.033331)
-		(width 0.25)
-		(layer "B.Cu")
-		(net "Net-(U2-IO17)")
-	)
-	(segment
-		(start 116.388299 97.175)
-		(end 117.938604 97.175)
-		(width 0.25)
-		(layer "B.Cu")
-		(net "Net-(U2-IO17)")
-	)
-	(segment
-		(start 120 95.5)
-		(end 119 95.5)
-		(width 0.25)
-		(layer "B.Cu")
-		(net "Net-(U2-IO17)")
+		(start 115.82 100.85)
+		(end 117.55 100.85)
+		(width 0.25)
+		(layer "B.Cu")
+		(net "Net-(U2-IO16)")
+	)
+	(segment
+		(start 121.695 88.985)
+		(end 122.275 88.985)
+		(width 0.25)
+		(layer "B.Cu")
+		(net "Net-(U2-IO16)")
+	)
+	(segment
+		(start 117.55 100.85)
+		(end 119.9 98.5)
+		(width 0.25)
+		(layer "B.Cu")
+		(net "Net-(U2-IO16)")
+	)
+	(segment
+		(start 114.3 99.33)
+		(end 115.82 100.85)
+		(width 0.25)
+		(layer "B.Cu")
+		(net "Net-(U2-IO16)")
 	)
 	(segment
 		(start 119.9 98.5)
-		(end 118.813604 97.413604)
+		(end 121.43 96.97)
 		(width 0.25)
 		(layer "B.Cu")
@@
 	)
 	(segment
-		(start 117.538604 94.675)
-		(end 116.388299 94.675)
+		(start 120.33 90.35)
+		(end 121.695 88.985)
 		(width 0.25)
 		(layer "B.Cu")
@@
 	)
 	(segment
-		(start 122.275 88.985)
-		(end 119.015 88.985)
+		(start 117 91)
+		(end 114.3 93.7)
 		(width 0.25)
 		(layer "B.Cu")
@@
 	)
 	(segment
-		(start 115.7 93.986701)
-		(end 115.7 92.3)
+		(start 114.3 93.7)
+		(end 114.3 99.33)
 		(width 0.25)
 		(layer "B.Cu")
@@
 	)
 	(segment
-		(start 115.7 92.3)
-		(end 116.681802 91.318198)
+		(start 121.43 93.41)
+		(end 120.33 92.31)
 		(width 0.25)
 		(layer "B.Cu")
@@
 	)
 	(segment
-		(start 118.813604 95.95)
-		(end 117.538604 94.675)
+		(start 121.43 96.97)
+		(end 121.43 93.41)
 		(width 0.25)
 		(layer "B.Cu")
@@
 	)
 	(segment
-		(start 116.388299 94.675)
-		(end 115.7 93.986701)
-		(width 0.25)
-		(layer "B.Cu")
-		(net "Net-(U2-IO16)")
-	)
-	(segment
-		(start 118.813604 97.413604)
-		(end 118.813604 95.95)
-		(width 0.25)
-		(layer "B.Cu")
-		(net "Net-(U2-IO16)")
-	)
-	(segment
-		(start 119.015 88.985)
-		(end 117 91)
-		(width 0.25)
-		(layer "B.Cu")
+		(start 120.33 92.31)
+		(end 120.33 90.35)
+		(width 0.25)
+		(layer "B.Cu")
